File: PDB.kicad_sch (KiCad schematic)
At the start: 35 parts, among them J0 XT90PW-M, J1 XT30PW-M, J2 XT30PW-M, J3 XT30PW-M, J4 XT30PW-M, J5 B2B-XH-A__LF__SN_, J6 B5B-XH-A, SW1 SW_Nidec_CAS-120A1, U1 TPS2490DGSR, U12 TPS54302

Commit message: ic's removed
Parts:
- removed C1: C, symbol Device:C
- removed C3: 0.01uF 100V, Capacitor_SMD:C_0603_1608Metric, symbol Device:C
- removed D1: SMC5K51A-M3/I, Diode_SMD:D_SMC, symbol Diode:1.5SMCxxA
- removed J5: B2B-XH-A__LF__SN_, B2B-XH-A__LF__SN_:JST_B2B-XH-A__LF__SN_, symbol B2B-XH-A__LF__SN_:B2B-XH-A__LF__SN_
- removed R1, R3, R4, R5, R6, R_Sense: R, symbol Device:R
- removed SW1: SW_Nidec_CAS-120A1, Button_Switch_SMD:Nidec_Copal_CAS-120A, symbol Switch:SW_Nidec_CAS-120A1
- removed U1: TPS2490DGSR, TPS2490DGSR:SOP50P490X110-10N, symbol TPS2490DGSR:TPS2490DGSR
- added J5, J7: Conn_01x01_Pin, Connector_Wire:SolderWirePad_1x01_SMD_3x6mm, symbol Connector:Conn_01x01_Pin
Connections:
- net GND: now also J7.1 (Pin_1)
- net VDD_5V_BRICK: now also J5.1 (Pin_1)
Other:
- note added: "LETS IMPLEMENT HARDWARE PRECHARGE CIRCUIT FUSE"
- moved on the sheet: J0

Commit message: new layout made
Parts:
- removed C2, C4, C5, C6: C, symbol Device:C
- removed J0: XT90PW-M, XT90PW-M:AMASS_XT90PW-M, symbol XT90PW-M:XT90PW-M
- removed J1, J2, J3, J4: XT30PW-M, XT30PW-M:AMASS_XT30PW-M, symbol XT30PW-M:XT30PW-M
- removed J6: B5B-XH-A, B5B-XH-A:JST_B5B-XH-A, symbol B5B-XH-A:B5B-XH-A
- added J1: XT60-M, XT60-M:AMASS_XT60-M, symbol XT60-M:XT60-M
- added J10, J11, J12, J13, J14, J6, J8, J9: Conn_01x01_Pin, Connector_Wire:SolderWirePad_1x01_SMD_3x6mm, symbol Connector:Conn_01x01_Pin
- R29: value 105k -> 100k
Connections:
- net GND: now also J1.N (NEG), J10.1 (Pin_1), J12.1 (Pin_1), J14.1 (Pin_1), J8.1 (Pin_1)
- net V_BAT: no longer names the net of C30.1, C31.1, R26.1, U12.3 (VIN)
- net V_BAT: now also J1.P (POS), J11.1 (Pin_1), J13.1 (Pin_1), J6.1 (Pin_1), J9.1 (Pin_1)
Other:
- note added: "DO WE NEED A FUSE"
- note removed: "LETS IMPLEMENT HARDWARE PRECHARGE CIRCUIT FUSE"
- moved on the sheet: C30, C31, C32, C33, C34, C35, J5, J7, L1, R26, R27, R28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

Commit message: up for review
Parts:
- L1: value 10u -> 10mH; footprint Inductor_SMD:L_0805_2012Metric -> footprints:IND_MWSA0603S_SNL
Other:
- moved on the sheet: C32, C33, C34, R28, R29, R30
