File: PDB.kicad_pcb (KiCad board)
At the start: 2 copper layers, 33.5 x 33.9 mm, 24 parts, among them J1 XT60-M, J10 Conn_01x01_Pin, J11 Conn_01x01_Pin, J12 Conn_01x01_Pin, J13 Conn_01x01_Pin, J14 Conn_01x01_Pin, J5 Conn_01x01_Pin, J6 Conn_01x01_Pin, J7 Conn_01x01_Pin, J8 Conn_01x01_Pin, J9 Conn_01x01_Pin, U12 TPS54302

Commit message: up for review
Parts:
- J10, J12, J14, J7, J8: moved to B.Cu
- L1: value 10u -> 10mH; footprint Inductor_SMD:L_0805_2012Metric -> footprints:IND_MWSA0603S_SNL
- moved J14 13.6 mm to (104.1, 75.8), turned to 180 degrees
- moved J7 13.2 mm to (104.6, 50.2), turned to 180 degrees
- moved J12 13.2 mm to (118.0, 50.2), turned to 180 degrees
- moved J8 13.1 mm to (117.8, 75.9), turned to 180 degrees
- moved R28 9.10 mm to (109.8, 61.0), turned to 180 degrees
- moved C30 4.65 mm to (110.9, 58.4), turned to -90 degrees
- moved C31 4.59 mm to (109.1, 58.7), turned to -90 degrees
- moved J10 4.50 mm to (117.9, 64.6), turned to 0 degrees
- moved C32 4.32 mm to (112.9, 60.0)
- moved C33 4.31 mm to (115.0, 60.0)
- moved J5 3.03 mm to (118.0, 63.3), turned to 180 degrees
- moved L1 2.48 mm to (110.9, 65.5), turned to 0 degrees
- moved C35 1.98 mm to (104.1, 66.8)
- moved C34 1.98 mm to (100.8, 60.6)
- moved R26 1.98 mm to (104.5, 61.0)
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Routing:
- net Net-(C34-Pad1): track 0.00 -> 10.9 mm
- net GND: track 0.00 -> 7.61 mm, vias 0 -> 40
- net Net-(U12-SW): track 0.00 -> 7.30 mm
- net Net-(U12-EN): track 0.00 -> 6.11 mm
- net Net-(U12-FB): track 0.00 -> 4.73 mm
- net Net-(J1-POS): track 0.00 -> 2.30 mm, vias 0 -> 36
- net Net-(U12-BOOT): track 0.00 -> 1.79 mm
- added copper zone on B.Cu, net GND
- added copper zone on F.Cu, net Net-(J1-POS)

Commit message: simulations pending
Parts:
- moved + 1.30 mm to (117.9, 64.6)
- renumbered J5 to +, J13 to +, J9 to +, J6 to +, J11 to +, J12 to -, J14 to -, J7 to -, J10 to -, J8 to -
Routing:
- net GND: track 7.61 -> 7.65 mm, vias 40 -> 76
- net Net-(J1-POS): vias 36 -> 72

Commit message: fusion simulation pending
Routing:
- net Net-(J1-POS): vias 72 -> 48
- net GND: vias 76 -> 52

Commit message: made board to 4 layer
Routing:
- added copper zone on In2.Cu, net GND
- added copper zone on In1.Cu, net Net-(J1-POS)
Other:
- copper layers 2 -> 4
Changed lines of the file:
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@@
 	(layers
 		(0 "F.Cu" signal)
+		(4 "In1.Cu" signal)
+		(6 "In2.Cu" signal)
 		(2 "B.Cu" signal)
 		(9 "F.Adhes" user "F.Adhesive")
@@
 		(43 "User.3" user)
 		(45 "User.4" user)
+		(47 "User.5" user)
 	)
 	(setup
+		(stackup
+			(layer "F.SilkS"
+				(type "Top Silk Screen")
+				(color "Black")
+			)
+			(layer "F.Paste"
+				(type "Top Solder Paste")
+			)
+			(layer "F.Mask"
+				(type "Top Solder Mask")
+				(thickness 0.01)
+			)
+			(layer "F.Cu"
+				(type "copper")
+				(thickness 0.035)
+			)
+			(layer "dielectric 1"
+				(type "prepreg")
+				(thickness 0.1)
+				(material "FR4")
+				(epsilon_r 4.5)
+				(loss_tangent 0.02)
+			)
+			(layer "In1.Cu"
+				(type "copper")
+				(thickness 0.035)
+			)
+			(layer "dielectric 2"
+				(type "core")
+				(thickness 1.24)
+				(material "FR4")
+				(epsilon_r 4.5)
+				(loss_tangent 0.02)
+			)
+			(layer "In2.Cu"
+				(type "copper")
+				(thickness 0.035)
+			)
+			(layer "dielectric 3"
+				(type "prepreg")
+				(thickness 0.1)
+				(material "FR4")
+				(epsilon_r 4.5)
+				(loss_tangent 0.02)
+			)
+			(layer "B.Cu"
+				(type "copper")
+				(thickness 0.035)
+			)
+			(layer "B.Mask"
+				(type "Bottom Solder Mask")
+				(thickness 0.01)
+			)
+			(layer "B.Paste"
+				(type "Bottom Solder Paste")
+			)
+			(layer "B.SilkS"
+				(type "Bottom Silk Screen")
+			)
+			(copper_finish "None")
+			(dielectric_constraints no)
+		)
 		(pad_to_mask_clearance 0)
 		(allow_soldermask_bridges_in_footprints no)
@@
 		(layer "Edge.Cuts")
 	)
+	(dimension
+		(type orthogonal)
+		(layer "Dwgs.User")
+		(pts
+			(xy 120.5 46.05) (xy 87.025 48.35)
+		)
+		(height -1.65)
+		(orientation 0)
+		(format
+			(prefix "")
+			(suffix "")
+			(units 3)
+			(units_format 0)
+			(precision 4)
+			(suppress_zeroes yes)
+		)
+		(style
+			(thickness 0.1)
+			(arrow_length 1.27)
+			(text_position_mode 0)
+			(arrow_direction outward)
+			(extension_height 0.58642)
+			(extension_offset 0.5)
+			(keep_text_aligned yes)
+		)
+		(gr_text "33.475"
+			(at 103.7625 43.79 0)
+			(layer "Dwgs.User")
+			(effects
+				(font
+					(size 0.5 0.5)
+					(thickness 0.11)
+				)
+			)
+		)
+	)
 	(segment
 		(start 112.925 59.05)
@@
 	)
 	(zone
-		(net "Net-(J1-POS)")
+		(net "VDD_5V_BRICK")
 		(layer "F.Cu")
-		(name "5v")
 		(hatch edge 0.5)
+		(priority 2)
 		(connect_pads yes
 			(clearance 0.5)
@@
 		(polygon
 			(pts
-				(xy 87.2 53.35) (xy 96.725 53.45) (xy 96.675 46.275) (xy 107.225 46.3) (xy 107.05 53.4) (xy 109.775 53.5)
-				(xy 109.775 46.375) (xy 120.2 46.275) (xy 120.275 79.75) (xy 109.675 79.775) (xy 109.65 72.825)
-				(xy 107.3 72.825) (xy 107.325 79.8) (xy 96.6 79.725) (xy 96.65 72.725) (xy 87.3 72.775)
+				(xy 109.464821 60.18787) (xy 120.043704 60.112072) (xy 120.096407 68.333522) (xy 109.516731 68.216624)
 			)
 		)
 	)
 	(zone
-		(net "VDD_5V_BRICK")
-		(layer "F.Cu")
+		(net "Net-(J1-POS)")
+		(layers "F.Cu" "In1.Cu")
+		(name "5v")
 		(hatch edge 0.5)
-		(priority 2)
 		(connect_pads yes
 			(clearance 0.5)
@@
 		(polygon
 			(pts
-				(xy 109.464821 60.18787) (xy 120.043704 60.112072) (xy 120.096407 68.333522) (xy 109.516731 68.216624)
+				(xy 87.2 53.35) (xy 96.725 53.45) (xy 96.675 46.275) (xy 107.225 46.3) (xy 107.05 53.4) (xy 109.775 53.5)
+				(xy 109.775 46.375) (xy 120.2 46.275) (xy 120.275 79.75) (xy 109.675 79.775) (xy 109.65 72.825)
+				(xy 107.3 72.825) (xy 107.325 79.8) (xy 96.6 79.725) (xy 96.65 72.725) (xy 87.3 72.775)
 			)
 		)
@@
 	(zone
 		(net "GND")
-		(layer "B.Cu")
+		(layers "B.Cu" "In2.Cu")
 		(hatch edge 0.5)
 		(priority 1)
